File: 555_Timer_Clock.kicad_pcb (KiCad board)
At the start: 2 copper layers, 39 x 25 mm, 13 parts, among them J2 CLK_Out, U1 ICM7555xB

Commit message: kiCad done
Parts:
- added J1: +5V, my_footprints:Terminal_Block_5mm, F.Cu at (102.5, 72.0)
- added SW1: Trigger, my_footprints:slide_switch_2.54mm, F.Cu at (121.5, 81.0)
- added SW2: RST, my_footprints:tact_switch_5mm, F.Cu at (111.0, 81.5)
Routing:
- net GND: track 0.00 -> 83.0 mm, vias 0 -> 2
- net /+5V: track 0.00 -> 38.8 mm
- net /Trigger: track 0.00 -> 36.0 mm
- net /CLK_Out: track 0.00 -> 26.9 mm, vias 0 -> 1
- net /RST: track 0.00 -> 19.4 mm
- net Net-(U1-DISCH): track 0.00 -> 12.9 mm
- net Net-(D1-K): track 0.00 -> 9.50 mm
- net Net-(U1-CONT): track 0.00 -> 7.46 mm
Other:
- board text removed: "NgiekNgiek"

Commit message: kiCad Done.
Parts:
- added G***: LOGO, ed:aottt, F.Cu at (104.2, 81.0)
